File: AFE.kicad_sch (KiCad schematic)
At the start: 18 parts, among them U8 LMH6881

Commit message: Fix SPI voltages, etc
Parts:
- removed R10: 15, symbol Device:R
- removed R38, R39: 50, symbol Device:R
- added C36, C37, C41: 100n, Capacitor_SMD:C_0603_1608Metric, symbol Device:C
- added C38, C39: 1u, Capacitor_SMD:C_0603_1608Metric, symbol Device:C
- added R19, R20, R21, R22: 10k, Resistor_SMD:R_0603_1608Metric, symbol Device:R
- added R26, R27: 7.5, Resistor_SMD:R_0603_1608Metric, symbol Device:R
- added U8: TXB0104RGY, Package_DFN_QFN:Texas_S-PVQFN-N14, symbol Logic_LevelTranslator:TXB0104RGY
- R23: renamed from R37; footprint (none) -> Resistor_SMD:R_0603_1608Metric
- renumbered C31 to C32, C32 to C33, C33 to C34, C34 to C35, C41 to C40, L4 to L3, L5 to L4, R8 to R24, R9 to R25, R12 to R28, R13 to R29, U8 to U9
Connections:
- net GND: now also U9.17 (SD), C36.2, C37.2, C41.2, U8.15 (Pad), U8.7 (GND)
- net MISO: now also R19.2, U8.4 (A3); no longer U9.4 (SDO)
- net MOSI: now also U8.5 (A4); no longer U9.3 (SDI)
- net SCLK: now also U8.3 (A2); no longer U9.15 (SCLK)
- net VCM: now also C41.1, R26.2, R27.1
- net ~{CS}: now also U8.2 (A1); no longer U9.16 (~{CS})
- net at L3.2, R24.2, R28.1: now also R26.1
- net at C40.1, L3.1, R24.1: now also C38.2; no longer U9.22 (OUTP)
- net at C40.2, L4.1, R25.1: now also C39.2; no longer U9.21 (OUTM)
- net at L4.2, R25.2, R29.1: now also R27.2
- net +3V3: now reaches U9.5 (SPI)
- net +3V3: now also C37.1, R20.1, R21.1, R22.1, U8.14 (VCCB)
- net OCM: no longer names the net of U9.2 (OCM)
- new net: C39.1, U9.21 (OUTM)
- new net: C38.1, U9.22 (OUTP)
- new net +1V8: C36.1, R19.1, U8.1 (VCCA), U8.8 (OE)
- new net A_~{CS}: R20.2, U8.13 (B1), U9.16 (~{CS})
- new net SCK: R21.2, U8.12 (B2), U9.15 (SCLK)
- new net SI: R22.2, U8.10 (B4), U9.3 (SDI)
- new net SO: U8.11 (B3), U9.4 (SDO)
- no-connect marks 2 -> 3
Other:
- moved on the sheet: C40, L3, L4, R24, R25, R28, R29

Commit message: Add footprints, fix voltage mismatches, add i2c bus to FT600
Parts:
- added C69, C70, C71, C72: 100n, Capacitor_SMD:C_0603_1608Metric, symbol Device:C
- U8: lcsc_id (none) -> C400708
- U9: lcsc_id (none) -> C701929
Connections:
- net +5V: now also C69.1, C70.1, C71.1, C72.1
- net GND: now also C69.2, C70.2, C71.2, C72.2

Commit message: Fix ferrite, etc
Parts:
- renumbered C32 to C37, C33 to C38, C34 to C39, C35 to C40, C36 to C41, C69 to C42, C37 to C43, C70 to C44, C71 to C45, C72 to C46, C38 to C47, C39 to C48, C40 to C49, C41 to C50, R19 to R21, R20 to R22, R21 to R23, R22 to R24, R23 to R25, R24 to R26, R25 to R27, R26 to R28, R27 to R29, R28 to R30, R29 to R31
