File: USB-3.kicad_sch (KiCad schematic)
At the start: 22 parts, among them J3 USB_C_Receptacle, U2 HD3SS3220, U3 FT600, Y1 30M

Commit message: Fix SPI voltages, etc
Parts:
- removed Y1: 30M, symbol Device:Crystal_GND23
- added C68: 1u, Capacitor_SMD:C_0603_1608Metric, symbol Device:C
- added Y2: ABM3-30MHZ-D2Y-T, symbol Device:Crystal
- C13, C14: value C -> 18p
- FB1: value FerriteBead -> BK0603HS330-T
- J2: renamed from J3; footprint (none) -> plib:USB-C-SMD_C49261591
- renumbered R6 to R10, R7 to R11, R2 to R6, R3 to R7, R4 to R8, R5 to R9, U2 to U4, U3 to U5
Connections:
- net +5V: now also C68.1
- net GND: now also C68.2
- net at C13.1, U5.17 (XO): now also Y2.1
- net at C14.1, U5.16 (XI): now also Y2.2
Other:
- moved on the sheet: C10

Commit message: Add footprints, fix voltage mismatches, add i2c bus to FT600
Parts:
- removed Y2: ABM3-30MHZ-D2Y-T, symbol Device:Crystal
- added Y2: ABM10-30MHZ-E20-T, Crystal:Crystal_SMD_2520-4Pin_2.5x2.0mm, symbol Device:Crystal_GND24
- C11, C12, C8, C9: footprint Capacitor_SMD:C_0603_1608Metric -> Capacitor_SMD:C_0402_1005Metric
- FB1: value BK0603HS330-T -> BLM15GG471SN1#
- U4: lcsc_id (none) -> C165155
- U5: lcsc_id (none) -> C5252722
Connections:
- net GND: now also Y2.2, Y2.4
- net at C8.1: now also J2.A2 (TX1+); no longer J2.A3 (TX1-)
- net at C11.1: now also J2.A3 (TX1-); no longer J2.A2 (TX1+)
- net i2c scl: now reaches U5.12 (GPIO0)
- net i2c sda: now reaches U5.13 (GPIO1)
- net at C14.1, U5.16 (XI): now also Y2.3
- net at C13.1, U5.17 (XO): now also Y2.1
- no-connect marks 13 -> 11
Other:
- moved on the sheet: C8, C9

Commit message: Fix ferrite, etc
Parts:
- FB1: value BLM15GG471SN1# -> BLM18PG121SN1D; footprint (none) -> Inductor_SMD:L_0603_1608Metric
- renumbered C7 to C11, C68 to C12, C8 to C13, C9 to C14, C11 to C15, C12 to C16, C10 to C17, C13 to C18, C14 to C19, C15 to C20, C16 to C21, C17 to C22, R8 to R10, R9 to R11, R10 to R12, R11 to R13, R6 to R8, R7 to R9
