File: fpga.kicad_sch (KiCad schematic)
At the start: 27 parts, among them J4 FPGA PROG, U4 ICE40UP5K-SG48ITR, U6 W25Q128JVS

Commit message: Fix SPI voltages, etc
Parts:
- renumbered C20 to C18, C18 to C19, C19 to C20, C69 to C24, C24 to C25, C25 to C26, C26 to C27, C27 to C28, C28 to C29, C29 to C30, C30 to C31, J4 to J3, R29 to R12, R26 to R13, R31 to R14, R30 to R15, R27 to R16, R28 to R17, R32 to R18, U4 to U6, U6 to U7

Commit message: Add footprints, fix voltage mismatches, add i2c bus to FT600
Parts:
- J3: footprint (none) -> Connector_PinHeader_2.54mm:PinHeader_1x06_P2.54mm_Vertical
- U6: lcsc_id (none) -> C2678152
- U7: lcsc_id (none) -> C97521
Changed lines of the file:
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@@
 			)
 		)
-		(property "lcsc_id" ""
+		(property "lcsc_id" "C2678152"
 			(at 43.18 119.38 0)
 			(effects
@@
 			)
 		)
-		(property "lcsc_id" ""
+		(property "lcsc_id" "C2678152"
 			(at 45.72 175.26 0)
 			(effects
@@
 			)
 		)
-		(property "lcsc_id" ""
+		(property "lcsc_id" "C97521"
 			(at 177.8 83.82 0)
 			(effects
@@
 			)
 		)
-		(property "Footprint" ""
+		(property "Footprint" "Connector_PinHeader_2.54mm:PinHeader_1x06_P2.54mm_Vertical"
 			(at 147.32 78.74 0)
 			(effects
@@
 			)
 		)
-		(property "lcsc_id" ""
+		(property "lcsc_id" "C2678152"
 			(at 45.72 54.61 0)
 			(effects
@@
 			)
 		)
-		(property "lcsc_id" ""
+		(property "lcsc_id" "C2678152"
 			(at 213.36 132.08 0)
 			(effects

Commit message: Fix ferrite, etc
Parts:
- renumbered C18 to C23, C19 to C24, C20 to C25, C21 to C26, C22 to C27, C23 to C28, C24 to C29, C25 to C30, C26 to C31, C27 to C32, C28 to C33, C29 to C34, C30 to C35, C31 to C36, R12 to R14, R13 to R15, R14 to R16, R15 to R17, R16 to R18, R17 to R19, R18 to R20
